Commit message: Update object pool and fix the reset scaling problem

File: assets/objects/ycb_objects_origin_at_center_vhacd/urdfs/ball.urdf (robot description, URDF)
Before this commit: robot ball, 1 links, 0 joints
Links:
- link ball: geometry collision mesh filename=meshes/ball/collision.obj; visual mesh filename=meshes/ball/textured.obj

File: assets/objects/ycb_objects_origin_at_center_vhacd/urdfs/cube.urdf (robot description, URDF)
Before this commit: robot object, 1 links, 0 joints
Links:
- link object: mass None -> .1; geometry collision mesh filename=meshes/cube/textured.obj scale=1. 1. 1.; visual mesh filename=meshes/cube/collision.obj scale=1. 1. 1.

File: assets/objects/ycb_objects_origin_at_center_vhacd/urdfs/cube_arrow.urdf (robot description, URDF)
Before this commit: robot object, 1 links, 0 joints
Links:
- link object: mass None -> .1

File: assets/objects/ycb_objects_origin_at_center_vhacd/urdfs/cuboid.urdf (robot description, URDF)
Before this commit: robot object, 1 links, 0 joints
Links:
- link object: mass None -> .1

File: assets/objects/ycb_objects_origin_at_center_vhacd/urdfs/mug.urdf (robot description, URDF)
Before this commit: robot mug, 1 links, 0 joints
Links:
- link mug: geometry collision mesh filename=../meshes/mug/collision.obj scale=0.01 0.01 0.01; visual mesh filename=../meshes/mug/textured.obj scale=0.01 0.01 0.01

File: assets/objects/ycb_objects_origin_at_center_vhacd/urdfs/pentagram.urdf (robot description, URDF)
Before this commit: robot object, 1 links, 0 joints
Links:
- link object: mass None -> .1; geometry collision mesh filename=meshes/pentagram/textured.obj scale=1. 1. 1.; visual mesh filename=meshes/pentagram/collision.obj scale=1. 1. 1.

File: assets/objects/ycb_objects_origin_at_center_vhacd/urdfs/potted_meat_can.urdf (robot description, URDF)
Before this commit: robot potted_meat_can, 1 links, 0 joints
Links:
- link baseLink: geometry collision mesh filename=../meshes/potted_meat_can/collision.obj; visual mesh filename=../meshes/potted_meat_can/textured.obj

File: assets/objects/ycb_objects_origin_at_center_vhacd/urdfs/tomato_soup_can.urdf (robot description, URDF)
Before this commit: robot tomato_soup_can, 1 links, 0 joints
Links:
- link baseLink: geometry collision mesh filename=../meshes/tomato_soup_can/collision.obj; visual mesh filename=../meshes/tomato_soup_can/textured.obj
