Commit message: RoboSensai Solver Training pipeline V0.1

File: assets/robots/franka_description/robots/franka_panda.urdf (robot description, URDF)
Before this commit: robot panda, 11 links, 10 joints
Links:
- added link panda_gripper_mid
Joints:
- added joint panda_gripper_mid: type fixed, parent panda_hand, child panda_gripper_mid, origin xyz=0 0 0.104 rpy=0 0 0, axis 0 0 0
